File: OctoPad.kicad_pcb (KiCad board)
At the start: 2 copper layers, 138.1 x 138.1 mm, 17 parts, among them U1 ProMicro

Commit message: 4/4/20 v2
Parts:
- added REF**: MountingHole_2.2mm_M2, MountingHole:MountingHole_2.2mm_M2, F.Cu at (367.5, 90.5)
- added REF**: MountingHole_2.2mm_M2, MountingHole:MountingHole_2.2mm_M2, F.Cu at (284.2, 54.8)
- added REF**: MountingHole_2.2mm_M2, MountingHole:MountingHole_2.2mm_M2, F.Cu at (248.4, 138.1)
- added REF**: MountingHole_2.2mm_M2, MountingHole:MountingHole_2.2mm_M2, F.Cu at (331.8, 173.8)
- added REF**: MountingHole_2.2mm_M2, MountingHole:MountingHole_2.2mm_M2, F.Cu at (135.7, 54.8)
- added REF**: MountingHole_2.2mm_M2, MountingHole:MountingHole_2.2mm_M2, F.Cu at (100.0, 138.1)
- added REF**: MountingHole_2.2mm_M2, MountingHole:MountingHole_2.2mm_M2, F.Cu at (183.4, 173.8)
- added REF**: MountingHole_2.2mm_M2, MountingHole:MountingHole_2.2mm_M2, F.Cu at (219.1, 90.5)
Other:
- board size 138.1 x 138.1 mm -> 286.6 x 138.1 mm
Changed lines of the file:
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@@
     (thickness 1.6)
     (drawings 6)
-    (tracks 108)
+    (tracks 106)
     (zones 0)
-    (modules 17)
+    (modules 25)
     (nets 31)
   )
@@
       (outputformat 1)
       (mirror false)
-      (drillshape 1)
+      (drillshape 0)
       (scaleselection 1)
-      (outputdirectory ""))
+      (outputdirectory "Gerbers/"))
   )
   (net 0 "")
@@
     (add_net ROW7)
   )
+  (module MountingHole:MountingHole_2.2mm_M2 (layer F.Cu)
+    (at 367.50625 90.4875)
+    (descr "Mounting Hole 2.2mm, no annular, M2")
+    (tags "mounting hole 2.2mm no annular m2")
+    (attr virtual)
+    (fp_text reference REF** (at 0 -3.2) (layer F.SilkS) hide
+      (effects (font (size 1 1) (thickness 0.15)))
+    )
+    (fp_text value MountingHole_2.2mm_M2 (at 0 3.2) (layer F.Fab)
+      (effects (font (size 1 1) (thickness 0.15)))
+    )
+    (fp_text user %R (at 0.3 0) (layer F.Fab)
+      (effects (font (size 1 1) (thickness 0.15)))
+    )
+    (fp_circle (center 0 0) (end 2.2 0) (layer Cmts.User) (width 0.15))
+    (fp_circle (center 0 0) (end 2.45 0) (layer F.CrtYd) (width 0.05))
+    (pad 1 np_thru_hole circle (at 0 0) (size 2.2 2.2) (drill 2.2) (layers *.Cu *.Mask))
+  )
+  (module MountingHole:MountingHole_2.2mm_M2 (layer F.Cu)
+    (at 284.1625 54.76875)
+    (descr "Mounting Hole 2.2mm, no annular, M2")
+    (tags "mounting hole 2.2mm no annular m2")
+    (attr virtual)
+    (fp_text reference REF** (at 0 -3.2) (layer F.SilkS) hide
+      (effects (font (size 1 1) (thickness 0.15)))
+    )
+    (fp_text value MountingHole_2.2mm_M2 (at 0 3.2) (layer F.Fab)
+      (effects (font (size 1 1) (thickness 0.15)))
+    )
+    (fp_circle (center 0 0) (end 2.45 0) (layer F.CrtYd) (width 0.05))
+    (fp_circle (center 0 0) (end 2.2 0) (layer Cmts.User) (width 0.15))
+    (fp_text user %R (at 0.3 0) (layer F.Fab)
+      (effects (font (size 1 1) (thickness 0.15)))
+    )
+    (pad 1 np_thru_hole circle (at 0 0) (size 2.2 2.2) (drill 2.2) (layers *.Cu *.Mask))
+  )
+  (module MountingHole:MountingHole_2.2mm_M2 (layer F.Cu)
+    (at 248.44375 138.1125)
+    (descr "Mounting Hole 2.2mm, no annular, M2")
+    (tags "mounting hole 2.2mm no annular m2")
+    (attr virtual)
+    (fp_text reference REF** (at 0 -3.2) (layer F.SilkS) hide
+      (effects (font (size 1 1) (thickness 0.15)))
+    )
+    (fp_text value MountingHole_2.2mm_M2 (at 0 3.2) (layer F.Fab)
+      (effects (font (size 1 1) (thickness 0.15)))
+    )
+    (fp_circle (center 0 0) (end 2.45 0) (layer F.CrtYd) (width 0.05))
+    (fp_circle (center 0 0) (end 2.2 0) (layer Cmts.User) (width 0.15))
+    (fp_text user %R (at 0.3 0) (layer F.Fab)
+      (effects (font (size 1 1) (thickness 0.15)))
+    )
+    (pad 1 np_thru_hole circle (at 0 0) (size 2.2 2.2) (drill 2.2) (layers *.Cu *.Mask))
+  )
+  (module MountingHole:MountingHole_2.2mm_M2 (layer F.Cu)
+    (at 331.7875 173.83125)
+    (descr "Mounting Hole 2.2mm, no annular, M2")
+    (tags "mounting hole 2.2mm no annular m2")
+    (attr virtual)
+    (fp_text reference REF** (at 0 -3.2) (layer F.SilkS) hide
+      (effects (font (size 1 1) (thickness 0.15)))
+    )
+    (fp_text value MountingHole_2.2mm_M2 (at 0 3.2) (layer F.Fab)
+      (effects (font (size 1 1) (thickness 0.15)))
+    )
+    (fp_circle (center 0 0) (end 2.45 0) (layer F.CrtYd) (width 0.05))
+    (fp_circle (center 0 0) (end 2.2 0) (layer Cmts.User) (width 0.15))
+    (fp_text user %R (at 0.3 0) (layer F.Fab)
+      (effects (font (size 1 1) (thickness 0.15)))
+    )
+    (pad 1 np_thru_hole circle (at 0 0) (size 2.2 2.2) (drill 2.2) (layers *.Cu *.Mask))
+  )
+  (module MountingHole:MountingHole_2.2mm_M2 (layer F.Cu)
+    (at 135.73125 54.76875)
+    (descr "Mounting Hole 2.2mm, no annular, M2")
+    (tags "mounting hole 2.2mm no annular m2")
+    (attr virtual)
+    (fp_text reference REF** (at 0 -3.2) (layer F.SilkS) hide
+      (effects (font (size 1 1) (thickness 0.15)))
+    )
+    (fp_text value MountingHole_2.2mm_M2 (at 0 3.2) (layer F.Fab)
+      (effects (font (size 1 1) (thickness 0.15)))
+    )
+    (fp_text user %R (at 0.3 0) (layer F.Fab)
+      (effects (font (size 1 1) (thickness 0.15)))
+    )
+    (fp_circle (center 0 0) (end 2.2 0) (layer Cmts.User) (width 0.15))
+    (fp_circle (center 0 0) (end 2.45 0) (layer F.CrtYd) (width 0.05))
+    (pad 1 np_thru_hole circle (at 0 0) (size 2.2 2.2) (drill 2.2) (layers *.Cu *.Mask))
+  )
+  (module MountingHole:MountingHole_2.2mm_M2 (layer F.Cu)
+    (at 100.0125 138.1125)
+    (descr "Mounting Hole 2.2mm, no annular, M2")
+    (tags "mounting hole 2.2mm no annular m2")
+    (attr virtual)
+    (fp_text reference REF** (at 0 -3.2) (layer F.SilkS) hide
+      (effects (font (size 1 1) (thickness 0.15)))
+    )
+    (fp_text value MountingHole_2.2mm_M2 (at 0 3.2) (layer F.Fab)
+      (effects (font (size 1 1) (thickness 0.15)))
+    )
+    (fp_text user %R (at 0.3 0) (layer F.Fab)
+      (effects (font (size 1 1) (thickness 0.15)))
+    )
+    (fp_circle (center 0 0) (end 2.2 0) (layer Cmts.User) (width 0.15))
+    (fp_circle (center 0 0) (end 2.45 0) (layer F.CrtYd) (width 0.05))
+    (pad 1 np_thru_hole circle (at 0 0) (size 2.2 2.2) (drill 2.2) (layers *.Cu *.Mask))
+  )
+  (module MountingHole:MountingHole_2.2mm_M2 (layer F.Cu)
+    (at 183.35625 173.83125)
+    (descr "Mounting Hole 2.2mm, no annular, M2")
+    (tags "mounting hole 2.2mm no annular m2")
+    (attr virtual)
+    (fp_text reference REF** (at 0 -3.2) (layer F.SilkS) hide
+      (effects (font (size 1 1) (thickness 0.15)))
+    )
+    (fp_text value MountingHole_2.2mm_M2 (at 0 3.2) (layer F.Fab)
+      (effects (font (size 1 1) (thickness 0.15)))
+    )
+    (fp_text user %R (at 0.3 0) (layer F.Fab)
+      (effects (font (size 1 1) (thickness 0.15)))
+    )
+    (fp_circle (center 0 0) (end 2.2 0) (layer Cmts.User) (width 0.15))
+    (fp_circle (center 0 0) (end 2.45 0) (layer F.CrtYd) (width 0.05))
+    (pad 1 np_thru_hole circle (at 0 0) (size 2.2 2.2) (drill 2.2) (layers *.Cu *.Mask))
+  )
+  (module MountingHole:MountingHole_2.2mm_M2 (layer F.Cu)
+    (at 219.075 90.4875)
+    (descr "Mounting Hole 2.2mm, no annular, M2")
+    (tags "mounting hole 2.2mm no annular m2")
+    (attr virtual)
+    (fp_text reference REF** (at 0 -3.2) (layer F.SilkS) hide
+      (effects (font (size 1 1) (thickness 0.15)))
+    )
+    (fp_text value MountingHole_2.2mm_M2 (at 0 3.2) (layer F.Fab)
+      (effects (font (size 1 1) (thickness 0.15)))
+    )
+    (fp_circle (center 0 0) (end 2.45 0) (layer F.CrtYd) (width 0.05))
+    (fp_circle (center 0 0) (end 2.2 0) (layer Cmts.User) (width 0.15))
+    (fp_text user %R (at 0.3 0) (layer F.Fab)
+      (effects (font (size 1 1) (thickness 0.15)))
+    )
+    (pad 1 np_thru_hole circle (at 0 0) (size 2.2 2.2) (drill 2.2) (layers *.Cu *.Mask))
+  )
   (module MX_Alps_Hybrid:MX-1U-NoLED (layer F.Cu)
     (at 218.28125 114.3 90)
@@
     )
   )
+  (gr_circle (center 307.975 114.3) (end 238.91875 112.7125) (layer Edge.Cuts) (width 0.05))
   (gr_text rev1 (at 159.54375 135.73125) (layer F.SilkS)
     (effects (font (size 1.5 1.5) (thickness 0.3)))
@@
   (gr_circle (center 159.54375 114.3) (end 90.4875 112.7125) (layer Edge.Cuts) (width 0.05))
   (gr_circle (center 159.54375 114.3) (end 189.70625 115.09375) (layer F.SilkS) (width 0.12))
-  (gr_circle (center 159.54375 114.3) (end 228.6 115.09375) (layer F.SilkS) (width 0.12))
   (segment (start 161.25 167.9175) (end 161.25 168.5375) (width 0.25) (layer F.Cu) (net 1))
   (segment (start 159.54375 166.21125) (end 161.29 167.9575) (width 0.25) (layer F.Cu) (net 1))
@@
   (segment (start 202.510526 77.355) (end 184.718026 59.5625) (width 0.25) (layer F.Cu) (net 17))
   (segment (start 202.510526 77.515128) (end 202.510526 77.355) (width 0.25) (layer F.Cu) (net 17))
-  (segment (start 135.476946 58.615156) (end 122.758878 71.333224) (width 0.25) (layer F.Cu) (net 17))
-  (segment (start 157.284844 58.615156) (end 135.476946 58.615156) (width 0.25) (layer F.Cu) (net 17))
-  (segment (start 157.7975 58.1025) (end 157.284844 58.615156) (width 0.25) (layer F.Cu) (net 17))
-  (segment (start 163.35375 58.1025) (end 157.7975 58.1025) (width 0.25) (layer F.Cu) (net 17))
   (segment (start 103.34625 135.789396) (end 119.32941 151.772556) (width 0.25) (layer F.Cu) (net 17))
   (segment (start 103.34625 110.49) (end 103.34625 135.789396) (width 0.25) (layer F.Cu) (net 17))
@@
   (segment (start 116.767279 77.701471) (end 116.767279 88.874312) (width 0.25) (layer F.Cu) (net 17))
   (segment (start 122.758878 71.709872) (end 116.767279 77.701471) (width 0.25) (layer F.Cu) (net 17))
+  (segment (start 135.989602 58.1025) (end 122.758878 71.333224) (width 0.25) (layer F.Cu) (net 17))
+  (segment (start 163.35375 58.1025) (end 135.989602 58.1025) (width 0.25) (layer F.Cu) (net 17))
   (segment (start 106.006025 84.986248) (end 105.034009 84.014232) (width 0.25) (layer B.Cu) (net 19))
   (segment (start 107.380663 84.986248) (end 106.006025 84.986248) (width 0.25) (layer B.Cu) (net 19))
